Commit message: add: EtherCAT/CANFD interface & fingertip tactile array sensor

File: dexhand_description/config/dexhand.ros2_control.xacro (robot description, xacro)
@@ -1,4 +1,9 @@
 <?xml version="1.0"?>
 <robot xmlns:xacro="http://www.ros.org/wiki/xacro">
+    <!-- 手势 gpio 只在实现了 do_gesture 的硬件接口上注入：Humble 版硬件接口把所有 gpio 当作
+         触觉区域处理，不导出 mode/gesture_id 命令接口，注入后 ResourceManager 会因找不到接口
+         而让整个硬件激活失败。默认按发行版判断，可用 use_gesture_gpio:=true/false 显式覆盖。 -->
+    <xacro:property name="ros_distro" value="$(optenv ROS_DISTRO jazzy)"/>
+    <xacro:arg name="use_gesture_gpio" default="${ros_distro != 'humble'}"/>
     <xacro:macro name="command_state_interface" params="name joint_limit init_position ">
         <joint name="${name}">
@@ -83,6 +88,25 @@
         </xacro:if>
     </xacro:macro>
+    <xacro:macro name="loop_gesture_interface" params="prefix:=^">
+        <xacro:if value="${prefix}">
+            <xacro:property name="pre" value="${prefix.pop(0)}"/>
+            <gpio name="${pre}do_gesture">
+                <!-- ros2_control 4.29 仅支持 double/bool；接口值仍严格遵循 uint8 语义。 -->
+                <command_interface name="mode" data_type="double">
+                    <!-- 1 = TOPIC：上电即按 topic 命令控制，无 IDLE 中间态 -->
+                    <param name="initial_value">1</param>
+                </command_interface>
+                <command_interface name="gesture_id" data_type="double">
+                    <param name="initial_value">0</param>
+                </command_interface>
+                <state_interface name="result" data_type="double">
+                    <param name="initial_value">0</param>
+                </state_interface>
+            </gpio>
+            <xacro:loop_gesture_interface/>
+        </xacro:if>
+    </xacro:macro>
     <xacro:macro name="dexhand_ros2_control" params="name initial_positions_file joint_limits_file use_gazebo:=false use_mock_dexhand:=false
-                                                     port_name:=/dev/dexhand hand_id:=0 baudrate:=1000000 timeout_ms:=200 prefix:=${['']}">
+                                                     port_name:=/dev/dexhand communicate:=RS485 hand_id:=0 baudrate:=1000000 timeout_ms:=200 gesture_timeout_ms:=5000 prefix:=${['']}">
         <xacro:property name="initial_positions" value="${xacro.load_yaml(initial_positions_file)['initial_positions']}"/>
         <xacro:property name="joint_limits" value="${xacro.load_yaml(joint_limits_file)['joint_limits']}"/>
@@ -118,8 +142,10 @@
                     <plugin>dexhand_hardware_interface/DexhandHardwareInterface</plugin>
                     <param name="joint_prefix">${joint_prefix}</param>
+                    <param name="communicate">${communicate}</param>
                     <param name="port_name">${port_name}</param>
                     <param name="hand_id">${hand_id}</param>
                     <param name="baudrate">${baudrate}</param>
                     <param name="timeout_ms">${timeout_ms}</param>
+                    <param name="gesture_timeout_ms">${gesture_timeout_ms}</param>
                 </hardware>
             </xacro:unless>
@@ -129,4 +155,9 @@
             <xacro:property name="tactile_names" value="${['THT0', 'FFT0', 'MFT0', 'RFT0', 'LFT0']}"/>
             <xacro:loop_tactile_interface items="${list(tactile_names)}" prefix="${list(prefix)}"/>
+            <!-- 手势 Action 使用的命令与结果接口。判断放在此处而非 loop_gesture_interface 内部：
+                 xacro 在递归宏里求值 arg/property 会爆栈（maximum recursion depth exceeded）。 -->
+            <xacro:if value="${xacro.arg('use_gesture_gpio')}">
+                <xacro:loop_gesture_interface prefix="${list(prefix)}"/>
+            </xacro:if>
         </ros2_control>
     </xacro:macro>

File: dexhand_description/urdf/dexhand.urdf.xacro (robot description, xacro)
@@ -3,8 +3,11 @@
     <xacro:arg name="use_left_hand" default="true" />
     <xacro:arg name="prefix" default=""/>
+    <xacro:arg name="dexhand_type" default="gs_s1" />
     <xacro:arg name="use_ros2_control" default="true" />
     <xacro:arg name="use_gazebo" default="false" />
     <xacro:arg name="use_mock_dexhand" default="false" />
     <xacro:arg name="port_name" default="/dev/dexhand" />
+    <xacro:arg name="communicate" default="RS485" />
+    <xacro:arg name="gesture_timeout_ms" default="5000" />
 <!-- construct pure URDF start -->
     <xacro:include filename="$(find dexhand_description)/urdf/dexhand_single_macro.xacro"/>
@@ -12,5 +15,6 @@
     <link name="world"/>
     <!-- dexhand -->
-    <xacro:dexhand_single_macro use_left_hand="$(arg use_left_hand)"
+    <xacro:dexhand_single_macro dexhand_type="$(arg dexhand_type)"
+                                use_left_hand="$(arg use_left_hand)"
                                 use_ros2_control="$(arg use_ros2_control)"
                                 use_gazebo="$(arg use_gazebo)"
@@ -18,4 +22,6 @@
                                 prefix="$(arg prefix)"
                                 port_name="$(arg port_name)"
+                                communicate="$(arg communicate)"
+                                gesture_timeout_ms="$(arg gesture_timeout_ms)"
                                 parent_link="world"
                                 joint_type="fixed">

File: dexhand_description/urdf/dexhand_macro.xacro (robot description, xacro)
@@ -3,6 +3,7 @@
     <!-- dexhand_macro = forearm + hand -->
     <!-- use_left_hand: select hand side -->
+    <!-- dexhand_type: gs_s1（V3） -->
     <!-- if use more than one dexhand, use prefix. such as "lh_" or "rh_" -->
-    <xacro:macro name="dexhand_macro" params="use_left_hand prefix:='' parent_link joint_type *origin">
+    <xacro:macro name="dexhand_macro" params="use_left_hand prefix:='' parent_link joint_type dexhand_type:='gs_s1' *origin">
         <!-- Constants for robot description -->
         <xacro:property name="joint_pi2" value="1.5708"/>
@@ -11,20 +12,21 @@
         <xacro:property name="joint_acc" value="2.0"/>
         <xacro:property name="joint_effort" value="0.1"/>
-        <!-- forearm -->
-        <!-- xacro:include filename="$(find dexhand_description)/urdf/forearm_macro_for_mujoco.xacro"/-->
-        <xacro:include filename="$(find dexhand_description)/urdf/forearm_macro.xacro"/>
+        <xacro:property name="left_palm_mount_yaw" value="${1.5708 if dexhand_type == 'gs_s2' else -1.5708}"/>
+        <!-- 每个版本目录提供同名宏 -->
+        <xacro:include filename="$(find dexhand_description)/urdf/${dexhand_type}/forearm_macro.xacro"/>
         <xacro:forearm_macro use_left_hand="${use_left_hand}" prefix="${prefix}" parent_link="${parent_link}" joint_type="${joint_type}">
             <xacro:insert_block name="origin"/>
         </xacro:forearm_macro>
+        <!-- 文件名和宏名一致，只通过 dexhand_type 选择版本目录。 -->
+        <xacro:include filename="$(find dexhand_description)/urdf/${dexhand_type}/left_hand_macro.xacro"/>
+        <xacro:include filename="$(find dexhand_description)/urdf/${dexhand_type}/right_hand_macro.xacro"/>
         <!-- left hand -->
         <xacro:if value="${use_left_hand}">
-            <xacro:include filename="$(find dexhand_description)/urdf/left_hand_macro.xacro"/>
             <xacro:left_hand_macro prefix="${prefix}" parent_link="${prefix}pmbase" joint_type="fixed">
-                <origin xyz="-0.0138 0 0.01485" rpy="0 0 -1.5708" />
+                <origin xyz="-0.0138 0 0.01485" rpy="0 0 ${left_palm_mount_yaw}" />
             </xacro:left_hand_macro>
         </xacro:if>
         <!-- right hand -->
         <xacro:unless value="${use_left_hand}">
-            <xacro:include filename="$(find dexhand_description)/urdf/right_hand_macro.xacro"/>
             <xacro:right_hand_macro prefix="${prefix}" parent_link="${prefix}pmbase" joint_type="fixed">
                 <origin xyz="-0.011315 0 0.01845" rpy="0 0 -1.5708" />

File: dexhand_description/urdf/dexhand_single_macro.xacro (robot description, xacro)
@@ -3,10 +3,12 @@
     <!-- 定义全局参数 -->
     <xacro:arg name="dexhand_initial_positions_file" default="$(find dexhand_description)/config/initial_positions.yaml" />
-    <xacro:arg name="dexhand_joint_limits_file" default="$(find dexhand_description)/config/joint_limits.yaml" />
+    <xacro:arg name="dexhand_joint_limits_file" default="" />
     <xacro:arg name="dexhand_link_configs_file" default="$(find dexhand_description)/config/link_configs.yaml" />
     <!-- Import materials used in urdf -->
     <xacro:include filename="$(find dexhand_description)/urdf/inc/common.materials.xacro"/>
     <!-- dexhand_single_macro 单只手的macro -->
-    <xacro:macro name="dexhand_single_macro" params="use_left_hand use_ros2_control:=false use_gazebo:=false use_mock_dexhand:=false prefix:='' port_name:=/dev/dexhand parent_link joint_type *origin">
+    <xacro:macro name="dexhand_single_macro" params="use_left_hand use_ros2_control:=false use_gazebo:=false use_mock_dexhand:=false prefix:='' port_name:=/dev/dexhand communicate:=RS485 gesture_timeout_ms:=5000 parent_link joint_type dexhand_type:='gs_s1' *origin">
+        <!-- 显式文件优先；未指定时使用本次宏调用所选版本的限位。 -->
+        <xacro:property name="joint_limits_file" value="${xacro.arg('dexhand_joint_limits_file') or '$(find dexhand_description)/config/' + dexhand_type + '/joint_limits.yaml'}" />
         <!-- Constants for robot description -->
         <xacro:property name="joint_pi2" value="1.5708"/>
@@ -17,5 +19,5 @@
         <!-- construct pure URDF start -->
         <xacro:include filename="$(find dexhand_description)/urdf/dexhand_macro.xacro"/>
-        <xacro:dexhand_macro use_left_hand="${use_left_hand}" prefix="${prefix}" parent_link="${parent_link}" joint_type="${joint_type}">
+        <xacro:dexhand_macro use_left_hand="${use_left_hand}" prefix="${prefix}" parent_link="${parent_link}" joint_type="${joint_type}" dexhand_type="${dexhand_type}">
             <xacro:insert_block name="origin"/>
         </xacro:dexhand_macro>
@@ -30,6 +32,8 @@
                 use_mock_dexhand="${use_mock_dexhand}"
                 initial_positions_file="$(arg dexhand_initial_positions_file)"
-                joint_limits_file="$(arg dexhand_joint_limits_file)"
+                joint_limits_file="${joint_limits_file}"
                 port_name="${port_name}"
+                communicate="${communicate}"
+                gesture_timeout_ms="${gesture_timeout_ms}"
                 prefix="${prefix_list}"
             />
@@ -40,10 +44,10 @@
             <xacro:dexhand_gazebo_attribute
                 link_configs_file="$(arg dexhand_link_configs_file)"
-                joint_limits_file="$(arg dexhand_joint_limits_file)"
+                joint_limits_file="${joint_limits_file}"
                 prefix="${prefix_list}"
             />
             <xacro:dexhand_gazebo_plugin
                 use_ros2_control="${use_ros2_control}"
-                joint_limits_file="$(arg dexhand_joint_limits_file)"
+                joint_limits_file="${joint_limits_file}"
                 prefix="${prefix_list}"
             />

File: dexhand_description/urdf/two_dexhand_as_individual.urdf.xacro (robot description, xacro)
@@ -5,4 +5,5 @@
     <xacro:arg name="use_gazebo" default="false" />
     <xacro:arg name="use_mock_left_dexhand" default="true" />
+    <xacro:arg name="dexhand_type" default="gs_s1" />
     <xacro:arg name="use_mock_right_dexhand" default="true" />
     <xacro:arg name="lh_prefix" default="lh_"/>
@@ -10,4 +11,6 @@
     <xacro:arg name="lh_port_name" default="/dev/ttyACM0"/>
     <xacro:arg name="rh_port_name" default="/dev/ttyACM1"/>
+    <xacro:arg name="lh_communicate" default="RS485"/>
+    <xacro:arg name="rh_communicate" default="RS485"/>
 <!-- construct pure URDF start -->
     <xacro:include filename="$(find dexhand_description)/urdf/dexhand_single_macro.xacro"/>
@@ -15,5 +18,6 @@
     <link name="world"/>
     <!-- left dexhand -->
-    <xacro:dexhand_single_macro use_left_hand="true"
+    <xacro:dexhand_single_macro dexhand_type="$(arg dexhand_type)"
+                                use_left_hand="true"
                                 use_ros2_control="$(arg use_ros2_control)"
                                 use_gazebo="$(arg use_gazebo)"
@@ -21,4 +25,5 @@
                                 prefix="$(arg lh_prefix)"
                                 port_name="$(arg lh_port_name)"
+                                communicate="$(arg lh_communicate)"
                                 parent_link="world"
                                 joint_type="fixed">
@@ -26,5 +31,6 @@
     </xacro:dexhand_single_macro>
     <!-- right dexhand -->
-    <xacro:dexhand_single_macro use_left_hand="false"
+    <xacro:dexhand_single_macro dexhand_type="$(arg dexhand_type)"
+                                use_left_hand="false"
                                 use_ros2_control="$(arg use_ros2_control)"
                                 use_gazebo="$(arg use_gazebo)"
@@ -32,4 +38,5 @@
                                 prefix="$(arg rh_prefix)"
                                 port_name="$(arg rh_port_name)"
+                                communicate="$(arg rh_communicate)"
                                 parent_link="world"
                                 joint_type="fixed">

File: dexhand_description/urdf/two_dexhand_as_whole.urdf.xacro (robot description, xacro)
@@ -5,6 +5,7 @@
     <xacro:arg name="use_gazebo" default="false" />
     <xacro:arg name="use_mock_dexhand" default="false" />
+    <xacro:arg name="dexhand_type" default="gs_s1" />
     <xacro:arg name="dexhand_initial_positions_file" default="$(find dexhand_description)/config/initial_positions.yaml" />
-    <xacro:arg name="dexhand_joint_limits_file" default="$(find dexhand_description)/config/joint_limits.yaml" />
+    <xacro:arg name="dexhand_joint_limits_file" default="$(find dexhand_description)/config/$(arg dexhand_type)/joint_limits.yaml" />
     <xacro:arg name="dexhand_link_configs_file" default="$(find dexhand_description)/config/link_configs.yaml" />
     <!-- Import materials used in urdf -->
@@ -18,9 +19,9 @@
     <link name="world"/>
     <!-- left dexhand -->
-    <xacro:dexhand_macro use_left_hand="true" prefix="$(arg lh_prefix)" parent_link="world" joint_type="fixed">
+    <xacro:dexhand_macro use_left_hand="true" prefix="$(arg lh_prefix)" parent_link="world" joint_type="fixed" dexhand_type="$(arg dexhand_type)">
         <origin xyz="0.5 0 0" rpy="0 0 0" />
     </xacro:dexhand_macro>
     <!-- right dexhand -->
-    <xacro:dexhand_macro use_left_hand="false" prefix="$(arg rh_prefix)" parent_link="world" joint_type="fixed">
+    <xacro:dexhand_macro use_left_hand="false" prefix="$(arg rh_prefix)" parent_link="world" joint_type="fixed" dexhand_type="$(arg dexhand_type)">
         <origin xyz="-0.5 0 0" rpy="0 0 0" />
     </xacro:dexhand_macro>
@@ -36,6 +37,6 @@
             use_gazebo="$(arg use_gazebo)"
             use_mock_dexhand="$(arg use_mock_dexhand)"
-            initial_positions_file="$(arg initial_positions_file)"
-            joint_limits_file="$(arg joint_limits_file)"
+            initial_positions_file="$(arg dexhand_initial_positions_file)"
+            joint_limits_file="$(arg dexhand_joint_limits_file)"
             prefix="${prefix_list}"
         />
@@ -45,11 +46,11 @@
         <xacro:include filename="$(find dexhand_description)/config/dexhand.gazebo.xacro"/>
         <xacro:dexhand_gazebo_attribute
-            link_configs_file="$(arg link_configs_file)"
-            joint_limits_file="$(arg joint_limits_file)"
+            link_configs_file="$(arg dexhand_link_configs_file)"
+            joint_limits_file="$(arg dexhand_joint_limits_file)"
             prefix="${prefix_list}"
         />
         <xacro:dexhand_gazebo_plugin
             use_ros2_control="$(arg use_ros2_control)"
-            joint_limits_file="$(arg joint_limits_file)"
+            joint_limits_file="$(arg dexhand_joint_limits_file)"
             prefix="${prefix_list}"
         />

Commit message: update: EtherCAT communication & do_gesture ROS action interface

File: dexhand_description/config/dexhand.ros2_control.xacro (robot description, xacro)
@@ -108,5 +108,5 @@
     </xacro:macro>
     <xacro:macro name="dexhand_ros2_control" params="name initial_positions_file joint_limits_file use_gazebo:=false use_mock_dexhand:=false
-                                                     port_name:=/dev/dexhand communicate:=RS485 hand_id:=0 baudrate:=1000000 timeout_ms:=200 gesture_timeout_ms:=5000 prefix:=${['']}">
+                                                     port_name:=/dev/dexhand communicate:=RS485 hand_id:=0 baudrate:=1000000 timeout_ms:=200 gesture_timeout_ms:=5000 debug:=false prefix:=${['']}">
         <xacro:property name="initial_positions" value="${xacro.load_yaml(initial_positions_file)['initial_positions']}"/>
         <xacro:property name="joint_limits" value="${xacro.load_yaml(joint_limits_file)['joint_limits']}"/>
@@ -148,4 +148,8 @@
                     <param name="timeout_ms">${timeout_ms}</param>
                     <param name="gesture_timeout_ms">${gesture_timeout_ms}</param>
+                    <!-- 调试开关：打开后 driver 输出详细日志，默认关闭 -->
+                    <param name="debug">${debug}</param>
+                    <!-- 设备身份 bridge topic：用相对名跟随 namespace 自动隔离（多手互不冲突），控制器按同名参数订阅 -->
+                    <param name="hand_info_topic">hand_info</param>
                 </hardware>
             </xacro:unless>

File: dexhand_description/urdf/dexhand.urdf.xacro (robot description, xacro)
@@ -10,4 +10,5 @@
     <xacro:arg name="communicate" default="RS485" />
     <xacro:arg name="gesture_timeout_ms" default="5000" />
+    <xacro:arg name="debug" default="false" />
 <!-- construct pure URDF start -->
     <xacro:include filename="$(find dexhand_description)/urdf/dexhand_single_macro.xacro"/>
@@ -24,4 +25,5 @@
                                 communicate="$(arg communicate)"
                                 gesture_timeout_ms="$(arg gesture_timeout_ms)"
+                                debug="$(arg debug)"
                                 parent_link="world"
                                 joint_type="fixed">

File: dexhand_description/urdf/dexhand_macro.xacro (robot description, xacro)
@@ -3,5 +3,5 @@
     <!-- dexhand_macro = forearm + hand -->
     <!-- use_left_hand: select hand side -->
-    <!-- dexhand_type: gs_s1（V3） -->
+    <!-- dexhand_type: gs_s1（V3）| gs_s2（V4） -->
     <!-- if use more than one dexhand, use prefix. such as "lh_" or "rh_" -->
     <xacro:macro name="dexhand_macro" params="use_left_hand prefix:='' parent_link joint_type dexhand_type:='gs_s1' *origin">
@@ -13,5 +13,5 @@
         <xacro:property name="joint_effort" value="0.1"/>
         <xacro:property name="left_palm_mount_yaw" value="${1.5708 if dexhand_type == 'gs_s2' else -1.5708}"/>
-        <!-- 每个版本目录提供同名宏 -->
+        <!-- 每个版本目录提供同名宏；gs_s2 当前保存 gs_s1 前臂的独立副本。 -->
         <xacro:include filename="$(find dexhand_description)/urdf/${dexhand_type}/forearm_macro.xacro"/>
         <xacro:forearm_macro use_left_hand="${use_left_hand}" prefix="${prefix}" parent_link="${parent_link}" joint_type="${joint_type}">

File: dexhand_description/urdf/dexhand_single_macro.xacro (robot description, xacro)
@@ -8,5 +8,5 @@
     <xacro:include filename="$(find dexhand_description)/urdf/inc/common.materials.xacro"/>
     <!-- dexhand_single_macro 单只手的macro -->
-    <xacro:macro name="dexhand_single_macro" params="use_left_hand use_ros2_control:=false use_gazebo:=false use_mock_dexhand:=false prefix:='' port_name:=/dev/dexhand communicate:=RS485 gesture_timeout_ms:=5000 parent_link joint_type dexhand_type:='gs_s1' *origin">
+    <xacro:macro name="dexhand_single_macro" params="use_left_hand use_ros2_control:=false use_gazebo:=false use_mock_dexhand:=false prefix:='' port_name:=/dev/dexhand communicate:=RS485 gesture_timeout_ms:=5000 debug:=false parent_link joint_type dexhand_type:='gs_s1' *origin">
         <!-- 显式文件优先；未指定时使用本次宏调用所选版本的限位。 -->
         <xacro:property name="joint_limits_file" value="${xacro.arg('dexhand_joint_limits_file') or '$(find dexhand_description)/config/' + dexhand_type + '/joint_limits.yaml'}" />
@@ -36,4 +36,5 @@
                 communicate="${communicate}"
                 gesture_timeout_ms="${gesture_timeout_ms}"
+                debug="${debug}"
                 prefix="${prefix_list}"
             />
