Commit message: add: sub_version 3 for gs_s1 series/model

File: dexhand_description/urdf/dexhand.urdf.xacro (robot description, xacro)
@@ -4,4 +4,5 @@
     <xacro:arg name="prefix" default=""/>
     <xacro:arg name="dexhand_type" default="gs_s1" />
+    <xacro:arg name="sub_version" default="original" />
     <xacro:arg name="use_ros2_control" default="true" />
     <xacro:arg name="use_gazebo" default="false" />
@@ -17,4 +18,5 @@
     <!-- dexhand -->
     <xacro:dexhand_single_macro dexhand_type="$(arg dexhand_type)"
+                                sub_version="$(arg sub_version)"
                                 use_left_hand="$(arg use_left_hand)"
                                 use_ros2_control="$(arg use_ros2_control)"

File: dexhand_description/urdf/dexhand_macro.xacro (robot description, xacro)
@@ -3,7 +3,8 @@
     <!-- dexhand_macro = forearm + hand -->
     <!-- use_left_hand: select hand side -->
-    <!-- dexhand_type: gs_s1（V3）| gs_s2（V4） -->
+    <!-- dexhand_type: gs_s1 | gs_s2 -->
+    <!-- sub_version: 1/2 keeps the existing asset set; 3 selects the new wrist -->
     <!-- if use more than one dexhand, use prefix. such as "lh_" or "rh_" -->
-    <xacro:macro name="dexhand_macro" params="use_left_hand prefix:='' parent_link joint_type dexhand_type:='gs_s1' *origin">
+    <xacro:macro name="dexhand_macro" params="use_left_hand prefix:='' parent_link joint_type dexhand_type:='gs_s1' sub_version:=1 *origin">
         <!-- Constants for robot description -->
         <xacro:property name="joint_pi2" value="1.5708"/>
@@ -12,23 +13,36 @@
         <xacro:property name="joint_acc" value="2.0"/>
         <xacro:property name="joint_effort" value="0.1"/>
-        <xacro:property name="left_palm_mount_yaw" value="${1.5708 if dexhand_type == 'gs_s2' else -1.5708}"/>
-        <!-- 每个版本目录提供同名宏；gs_s2 当前保存 gs_s1 前臂的独立副本。 -->
-        <xacro:include filename="$(find dexhand_description)/urdf/${dexhand_type}/forearm_macro.xacro"/>
+        <!-- Only the wrist implementation varies; both implementations keep the same macro interface. -->
+        <xacro:if value="${sub_version == 3}">
+            <xacro:include filename="$(find dexhand_description)/urdf/${dexhand_type}/sv_3/forearm_macro.xacro"/>
+        </xacro:if>
+        <xacro:unless value="${sub_version == 3}">
+            <xacro:include filename="$(find dexhand_description)/urdf/${dexhand_type}/forearm_macro.xacro"/>
+        </xacro:unless>
         <xacro:forearm_macro use_left_hand="${use_left_hand}" prefix="${prefix}" parent_link="${parent_link}" joint_type="${joint_type}">
             <xacro:insert_block name="origin"/>
         </xacro:forearm_macro>
-        <!-- 文件名和宏名一致，只通过 dexhand_type 选择版本目录。 -->
-        <xacro:include filename="$(find dexhand_description)/urdf/${dexhand_type}/left_hand_macro.xacro"/>
-        <xacro:include filename="$(find dexhand_description)/urdf/${dexhand_type}/right_hand_macro.xacro"/>
         <!-- left hand -->
         <xacro:if value="${use_left_hand}">
+            <xacro:include filename="$(find dexhand_description)/urdf/${dexhand_type}/left_hand_macro.xacro"/>
             <xacro:left_hand_macro prefix="${prefix}" parent_link="${prefix}pmbase" joint_type="fixed">
-                <origin xyz="-0.0138 0 0.01485" rpy="0 0 ${left_palm_mount_yaw}" />
+                <xacro:if value="${sub_version == 3}">
+                    <origin xyz="0 0 0.01485" rpy="0 0 -1.5708" />
+                </xacro:if>
+                <xacro:unless value="${sub_version == 3}">
+                        <origin xyz="-0.0138 0 0.01485" rpy="0 0 -1.5708" />
+                </xacro:unless>
             </xacro:left_hand_macro>
         </xacro:if>
         <!-- right hand -->
         <xacro:unless value="${use_left_hand}">
+            <xacro:include filename="$(find dexhand_description)/urdf/${dexhand_type}/right_hand_macro.xacro"/>
             <xacro:right_hand_macro prefix="${prefix}" parent_link="${prefix}pmbase" joint_type="fixed">
-                <origin xyz="-0.011315 0 0.01845" rpy="0 0 -1.5708" />
+                <xacro:if value="${sub_version == 3}">
+                    <origin xyz="0.0024852 0 0.01845" rpy="0 0 -1.5708" />
+                </xacro:if>
+                <xacro:unless value="${sub_version == 3}">
+                        <origin xyz="-0.011315 0 0.01845" rpy="0 0 -1.5708" />
+                </xacro:unless>
             </xacro:right_hand_macro>
         </xacro:unless>

File: dexhand_description/urdf/dexhand_single_macro.xacro (robot description, xacro)
@@ -8,5 +8,5 @@
     <xacro:include filename="$(find dexhand_description)/urdf/inc/common.materials.xacro"/>
     <!-- dexhand_single_macro 单只手的macro -->
-    <xacro:macro name="dexhand_single_macro" params="use_left_hand use_ros2_control:=false use_gazebo:=false use_mock_dexhand:=false prefix:='' port_name:=/dev/dexhand communicate:=RS485 gesture_timeout_ms:=5000 debug:=false parent_link joint_type dexhand_type:='gs_s1' *origin">
+    <xacro:macro name="dexhand_single_macro" params="use_left_hand use_ros2_control:=false use_gazebo:=false use_mock_dexhand:=false prefix:='' port_name:=/dev/dexhand communicate:=RS485 gesture_timeout_ms:=5000 debug:=false parent_link joint_type dexhand_type:='gs_s1' sub_version:='original' *origin">
         <!-- 显式文件优先；未指定时使用本次宏调用所选版本的限位。 -->
         <xacro:property name="joint_limits_file" value="${xacro.arg('dexhand_joint_limits_file') or '$(find dexhand_description)/config/' + dexhand_type + '/joint_limits.yaml'}" />
@@ -19,5 +19,5 @@
         <!-- construct pure URDF start -->
         <xacro:include filename="$(find dexhand_description)/urdf/dexhand_macro.xacro"/>
-        <xacro:dexhand_macro use_left_hand="${use_left_hand}" prefix="${prefix}" parent_link="${parent_link}" joint_type="${joint_type}" dexhand_type="${dexhand_type}">
+        <xacro:dexhand_macro use_left_hand="${use_left_hand}" prefix="${prefix}" parent_link="${parent_link}" joint_type="${joint_type}" dexhand_type="${dexhand_type}" sub_version="${sub_version}">
             <xacro:insert_block name="origin"/>
         </xacro:dexhand_macro>

File: dexhand_description/urdf/two_dexhand_as_individual.urdf.xacro (robot description, xacro)
@@ -6,4 +6,5 @@
     <xacro:arg name="use_mock_left_dexhand" default="true" />
     <xacro:arg name="dexhand_type" default="gs_s1" />
+    <xacro:arg name="sub_version" default="original" />
     <xacro:arg name="use_mock_right_dexhand" default="true" />
     <xacro:arg name="lh_prefix" default="lh_"/>
@@ -19,4 +20,5 @@
     <!-- left dexhand -->
     <xacro:dexhand_single_macro dexhand_type="$(arg dexhand_type)"
+                                sub_version="$(arg sub_version)"
                                 use_left_hand="true"
                                 use_ros2_control="$(arg use_ros2_control)"
@@ -32,4 +34,5 @@
     <!-- right dexhand -->
     <xacro:dexhand_single_macro dexhand_type="$(arg dexhand_type)"
+                                sub_version="$(arg sub_version)"
                                 use_left_hand="false"
                                 use_ros2_control="$(arg use_ros2_control)"

File: dexhand_description/urdf/two_dexhand_as_whole.urdf.xacro (robot description, xacro)
@@ -6,4 +6,5 @@
     <xacro:arg name="use_mock_dexhand" default="false" />
     <xacro:arg name="dexhand_type" default="gs_s1" />
+    <xacro:arg name="sub_version" default="original" />
     <xacro:arg name="dexhand_initial_positions_file" default="$(find dexhand_description)/config/initial_positions.yaml" />
     <xacro:arg name="dexhand_joint_limits_file" default="$(find dexhand_description)/config/$(arg dexhand_type)/joint_limits.yaml" />
@@ -19,9 +20,9 @@
     <link name="world"/>
     <!-- left dexhand -->
-    <xacro:dexhand_macro use_left_hand="true" prefix="$(arg lh_prefix)" parent_link="world" joint_type="fixed" dexhand_type="$(arg dexhand_type)">
+    <xacro:dexhand_macro use_left_hand="true" prefix="$(arg lh_prefix)" parent_link="world" joint_type="fixed" dexhand_type="$(arg dexhand_type)" sub_version="$(arg sub_version)">
         <origin xyz="0.5 0 0" rpy="0 0 0" />
     </xacro:dexhand_macro>
     <!-- right dexhand -->
-    <xacro:dexhand_macro use_left_hand="false" prefix="$(arg rh_prefix)" parent_link="world" joint_type="fixed" dexhand_type="$(arg dexhand_type)">
+    <xacro:dexhand_macro use_left_hand="false" prefix="$(arg rh_prefix)" parent_link="world" joint_type="fixed" dexhand_type="$(arg dexhand_type)" sub_version="$(arg sub_version)">
         <origin xyz="-0.5 0 0" rpy="0 0 0" />
     </xacro:dexhand_macro>
